Commit message: collision body is simplified

File: assets/robots/dodo/dodobot_v3/urdf/dodobot_v3_1.urdf (robot description, URDF)
Before this commit: robot dodobot_v3, 9 links, 8 joints
Links:
- link body_link: geometry collision box size=0.21 0.26 0.22; visual mesh filename=package://dodobot_v3/meshes/body_link.STL
- link left_link_1: geometry collision capsule length=0.09 radius=0.026; visual mesh filename=package://dodobot_v3/meshes/left_link_1.STL
- link left_link_2: geometry collision capsule length=0.185 radius=0.03; visual mesh filename=package://dodobot_v3/meshes/left_link_2.STL
- link left_link_3: geometry collision capsule length=0.175 radius=0.03; visual mesh filename=package://dodobot_v3/meshes/left_link_3.STL
- link left_link_4: geometry collision box size=0.06 0.095 0.034; visual mesh filename=package://dodobot_v3/meshes/left_link_4.STL
- link right_link_1: geometry collision capsule length=0.09 radius=0.026; visual mesh filename=package://dodobot_v3/meshes/right_link_1.STL
- link right_link_2: geometry collision capsule length=0.18 radius=0.03; visual mesh filename=package://dodobot_v3/meshes/right_link_2.STL
- link right_link_3: geometry collision capsule length=0.175 radius=0.03; visual mesh filename=package://dodobot_v3/meshes/right_link_3.STL
- link right_link_4: geometry collision box size=0.06 0.095 0.034; visual mesh filename=package://dodobot_v3/meshes/right_link_4.STL

Commit message: edited values of simplified collision body

File: assets/robots/dodo/dodobot_v3/urdf/dodobot_v3_1.urdf (robot description, URDF)
Before this commit: robot dodobot_v3, 9 links, 8 joints
Links:
- link body_link: geometry collision box size=0.21 0.26 0.24; visual mesh filename=package://dodobot_v3/meshes/body_link.STL
