Commit message: changed urdf files, dodo.urdf is default

File: assets/robots/dodo/dodobot_v3/urdf/dodobot_v3_2.urdf (robot description, URDF)
Before this commit: robot dodobot_v3, 9 links, 8 joints
Joints:
- joint left_joint_2: axis 0 0 -1 -> 0 0 1
- joint right_joint_1: axis 0 0 1 -> 0 0 -1

File: assets/robots/dodo/dodobot_v3/urdf/dodobot_v3_3.urdf (robot description, URDF)
Before this commit: robot dodobot_v3, 9 links, 8 joints
Links:
- added link base_link
- link body_link: geometry collision box size=0.21 0.29 0.1825; visual mesh filename=package://dodobot_v3/meshes/body_link.STL
Joints:
- added joint base_to_body: type fixed, parent base_link, child body_link, origin xyz=0 0 0 rpy=0 0 -1.5708
- joint left_joint_1: axis 0 0 1 -> 0 0 -1
